File: radiosonde_lite_final.sch (EAGLE design)
At the start: 86 parts, among them IC1 NEO-M8, J1 10104110-0001LF, J2 AFC01-S24FCA-00, Q4 MMBT3904, Q5 MMBT3904, U1 BMP280, U2 SHT40-AD1B-R2, U3 VGDD79S433N0SA, U4 ESP32-WROOM-32D-N8, U5 ME6211C12M5G-N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

Commit message: fin
Parts:
- removed C14, C16, C18: 0.1uF, ruark2:0603_CAPACITOR
- removed R10, R11: 47, ruark2:0402_RESISTOR
- removed R12, R13, R14, R15, R16, R17, R19, R24, R26: 10, ruark2:0402_RESISTOR
- removed U5: ME6211C12M5G-N, ruark2:ME6211C12M5G-N
- added ANT3: ANT-916-HETH, ruark2:ANT-916-HETH
- added CR2, CR3: RED, ruark2:150060RS75000
- added J3: CONUFL001-SMD, ruark2:CONUFL001-SMD
- added L1: SEL, ruark2:0402_INDUCTOR
- C1: value 10uF -> DNP; device ruark2:0603_CAPACITOR -> ruark2:0402_CAPACITOR
- C11, C12, C13, C2, C3, C6, C7: device ruark2:0603_CAPACITOR -> ruark2:0402_CAPACITOR
- C15: value 0.1uF -> 10uF
- C4, C5, C8: value 10uF -> 0.1uF; device ruark2:0603_CAPACITOR -> ruark2:0402_CAPACITOR
- C9: value 0.1uF -> DNP; device ruark2:0603_CAPACITOR -> ruark2:0402_CAPACITOR
- J2: value AFC01-S24FCA-00 -> CONUFL001-SMD; device ruark2:AFC01-S24FCA-00 -> ruark2:CONUFL001-SMD
- R1: value 1k -> 10; device ruark2:0603_RESISTOR -> ruark2:0402_RESISTOR
- R6, R7: value 10 -> 10k
- U7: value XC6206-2.8V -> AT2659; device ruark2:XC6206-2.8V -> ruark2:AT2659
Connections:
- removed net CAM_RST: J2.RESET, R24.2
- removed net CSI_D0: J2.D2, R6.2
- removed net CSI_D1: J2.D3, R19.1
- removed net CSI_D2: J2.D4, R17.1
- removed net CSI_D3: J2.D5, R2.2
- removed net CSI_D4: J2.D6, R16.1
- removed net CSI_D5: J2.D7, R4.2
- removed net CSI_D6: J2.D8, R26.1
- removed net CSI_D7: J2.D9, R15.2
- removed net CSI_HSYNC: J2.HS, R7.2
- removed net CSI_MCLK: J2.MCLK, R10.2
- removed net CSI_PCLK: J2.PCLK, R11.2
- removed net CSI_VSYNC: J2.VS, R5.2
- removed net N$16: R4.1, U4.IO18
- removed net N$17: R15.1, U4.IO19
- removed net N$18: R11.1, U4.IO21
- removed net N$22: R7.1, U4.IO26
- removed net N$23: R10.1, U4.IO27
- removed net N$3: R24.1, U4.IO4
- removed net N$36: R17.2, U4.IO34
- removed net N$37: R19.2, U4.IO35
- removed net N$8: C7.1, C8.1, J2.AVDD, U7.OUT
- new net N$26: C2.1, IC1.9_VCC_RF, R1.1
- new net N$30: C12.2, J2.RF
- new net N$31: IC1.11_RF_IN, J3.RF, U7.RF_OUT
- net +3V3: now also C3.1, C4.1, C7.1, CR2.A; no longer C1.1, C14.1, C16.1, C18.1, C2.1, J2.DOVDD, U5.EN, U5.IN, U7.IN
- net GND: now also J2.GND, J3.GND, R6.1, R7.1; no longer C1.2, C12.2, C14.2, C16.2, C18.2, J2.AGND, J2.DGND, R1.1, U5.GND
- net GPIO36: no longer R26.2
- net GPIO39: no longer R16.2
- net GPS_VCC_RF: now also C8.1, R1.2, U7.EN, U7.VS; no longer C9.1, IC1.9_VCC_RF
- net HSPI_CLK: now also R2.2; no longer R12.2
- net HSPI_CS: now also R5.2; no longer R3.2
- net HSPI_MISO: now also R3.2; no longer R13.2
- net HSPI_MOSI: now also R4.2; no longer R14.2
- net N$1: now also R3.1; no longer R13.1
- net N$11: now also ANT3.P$1
- net N$12: now also CR3.K, R7.2; no longer R6.1, U4.IO32
- net N$13: now also R5.1; no longer R3.1
- net N$14: now also C1.1, C9.1; no longer IC1.11_RF_IN
- net N$19: no longer R5.1
- net N$29: now also R2.1; no longer R12.1
- net N$4: now also C1.2, L1.P$1; no longer J2.PWDN, R1.2
- net N$6: now also L1.P$2, U7.RF_IN; no longer C3.1, C4.1, J2.DVDD, U5.OUT
- net N$7: now also CR2.K, R6.2; no longer R2.1, U4.IO5
- net N$9: now also R4.1; no longer R14.1
- net NEO_PPS: now also CR3.A
- net SCL: no longer J2.SCL
- net SDA: no longer J2.SDA
Other:
- note added: "Trace impedance assumes GCWG 7.5m gap on 0.8mm substrate per JLC calculator for 50 Ohm trace."
- note added: "VGdd79S915N0S1 for 915 MHz"
- note removed: "Address 0x60 for I2C Read Address 0x61 for I2C Write"
- note removed: "Pinout and ESP32 pin selection based on this: https://docs.m5stack.com/en/unit/unit_cam"
- moved on the sheet: ANT1, C1, C11, C12, C13, C15, C17, C2, C20, C3, C4, C5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
