File: radiosonde_lite_final.brd (EAGLE design)
At the start: 94 x 50.8 mm, 76 parts, among them IC1 NEO-M8, J1 10104110-0001LF, J2 CONUFL001-SMD, J3 CONUFL001-SMD, Q4 MMBT3904, Q5 MMBT3904, U1 BMP280, U2 SHT40-AD1B-R2, U3 VGDD79S433N0SA, U4 ESP32-WROOM-32D-N8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

Commit message: update
Parts:
- removed Q4, Q5: MMBT3904, ruark2a:SOT23-3_CENTERED
- removed R22, R23: 10k, ruark2:R0402
- removed R25: 1k, ruark2:0603
- removed R29: DNP, ruark2:R0402
- removed R30, R34: 10, ruark2:R0402
- added C14, C16: 0.1uF, ruark2:0402_INDUCTOR
- added CR4: RED, ruark2:0603_DIODE
- added JP3: (no value), pinhead:1X04
- added R10, R11, R12, R15, R16: 10, ruark2:R0402
- added R14: 10k, ruark2:R0402
- added R17: 1k, ruark2:R0402
- C1: value DNP -> 220pF
- C8: value 0.1uF -> 22nF
- L1: value SEL -> 6.8nH
- R8: value 10 -> 1k
- moved R36 49.4 mm to (40.1, 6.60)
- moved R35 31.6 mm to (42.9, 6.60)
- moved R21 29.2 mm to (56.9, 27.9), turned to 90 degrees
- moved R32 26.2 mm to (48.5, 27.9), turned to 270 degrees
- moved R5 22.9 mm to (55.6, 27.9), turned to 270 degrees
- moved CR1 22.6 mm to (46.7, 27.4)
- moved R4 21.4 mm to (49.8, 27.9), turned to 270 degrees
- moved R3 20.6 mm to (45.0, 27.9), turned to 270 degrees
- moved R2 17.3 mm to (43.4, 27.9), turned to 270 degrees
- moved R20 10.9 mm to (38.4, 13.2)
- moved R8 6.10 mm to (40.4, 42.9)
- moved JP1 1.27 mm to (70.9, 41.7)
- moved C4 0.18 mm to (42.9, 8.64)
- moved C3 0.13 mm to (42.9, 9.91)
- renumbered R33 to R13
Connections:
- removed net BUSY: R30.2, U3.11
- removed net DIO1: R13.2, R29.2, U3.10
- removed net DTR: JP1.3, Q5.2, R22.2
- removed net HSPI_CLK: R2.2, U3.4
- removed net HSPI_CS: R5.2, U3.5
- removed net HSPI_MISO: R3.2, U3.2
- removed net HSPI_MOSI: R4.2, U3.3
- removed net N$21: R8.1, U4.10
- removed net N$24: Q4.1, R22.1
- removed net N$27: Q5.1, R23.1
- removed net RTS: JP1.2, Q4.2, R23.2
- new net LED1: CR1.A, R3.2
- new net LED2: CR4.A, R4.2
- new net N$16: R12.1, U4.29
- new net N$17: R13.1, U4.26
- new net N$18: CR4.K, R14.2
- new net N$3: R10.1, U4.30
- new net N$8: R11.1, U4.31
- new net RADIO_BUSY: R15.1, U3.11
- new net RADIO_DIO1: R16.1, U3.10
- new net RADIO_MISO: R11.2, U3.2
- new net RADIO_MOSI: R9.2, U3.3
- new net RADIO_SCK: R10.2, U3.4
- new net RADIO_SS: R12.2, U3.5
- net +3V3: now also C14.P$1, C16.P$1, JP3.2, R17.2, R8.2; no longer R25.2
- net EN: now also JP1.3, R8.1; no longer Q4.3, R25.1
- net GND: now also C14.P$2, C16.P$2, JP3.1, R14.1
- net IO0: now also JP1.2, R17.1; no longer Q5.3, R13.1
- net N$19: now also R15.2, U4.6; no longer U4.36
- net N$28: no longer CR1.A, R34.1
- net N$5: now also R16.2, U4.7; no longer R29.1, R30.1, U4.9
- net RADIO_RST: now also R2.2; no longer R34.2
- net SCL: now also JP3.3, R5.2; no longer R9.2
- net SDA: now also JP3.4, R13.2; no longer R8.2
Routing:
- net RADIO_MOSI: track 0.00 -> 73.1 mm, vias 0 -> 2
- net DIO1: track 71.9 -> 0.00 mm, vias 2 -> 0
- net RADIO_MISO: track 0.00 -> 56.0 mm, vias 0 -> 2
- net RADIO_SCK: track 0.00 -> 52.8 mm, vias 0 -> 2
- net RADIO_SS: track 0.00 -> 50.7 mm, vias 0 -> 2
- net RADIO_BUSY: track 0.00 -> 46.3 mm
- net BUSY: track 43.7 -> 0.00 mm
- net RADIO_DIO1: track 0.00 -> 43.2 mm
- net N$28: track 44.5 -> 4.28 mm
- net N$13: track 32.4 -> 4.28 mm, vias 2 -> 0
- net N$1: track 27.1 -> 4.26 mm, vias 2 -> 0
- net N$9: track 26.3 -> 3.58 mm
- net RADIO_RST: track 8.33 -> 30.5 mm
- net N$29: track 25.3 -> 7.14 mm
- net SDA: track 86.3 -> 103.6 mm, vias 4 -> 0
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Other:
- outline, holes or cut-outs redrawn
- board text added: "3V3"
- board text added: "EN"
- board text added: "IO0"
- board text added: "SCL"
- board text added: "SDA"
- board text added: "TX"
- board text removed: "DTR"
- board text removed: "RTS"
- board text removed: "T"
